File: Nemesis-MixSigPCB.kicad_pcb (KiCad board)
At the start: 4 copper layers, 50 x 60 mm, 113 parts, among them J200 USB_C_Receptacle_USB2.0, J201 2x5 1.27mm, J300 031-5640-1010, J400 031-5640-1010, U100 HT7533-1, U101 TLV62569DBV, U102 MCP6001T-E/OT, U200 STM32F103CBT6, U201 USBLC6-2SC6, U300 MCP6001T-E/OT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

Commit message: AddedManufactureFiles
Routing:
- net GND: vias 78 -> 227
Other:
- board text added: "20 Hz < BW < 20kHz"
- board text added: "IN"
- board text added: "NEMESIS Signal Analyser and Generator"
- board text added: "ON"
- board text added: "OUT"
- board text added: "SWD"
- board text added: "USB"
